File: LED-JK3030.kicad_pcb (KiCad board)
At the start: 2 copper layers, 25 x 40 mm, 11 parts, among them J1 +, J2 -

Commit message: Final v1.0 layout
Other:
- board size 25 x 40 mm -> 24 x 40 mm
Changed lines of the file:
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@@
     (links 7)
     (no_connects 0)
-    (area 130.466667 79.424999 160.533333 119.575001)
+    (area 130.466667 79.424999 160.533333 119.583993)
     (thickness 1.6)
     (drawings 11)
@@
   (page A4)
   (title_block
-    (title "WiLED JK3030 LED array")
-    (date 2018-07-01)
-    (rev 1.0)
-    (company "Sean Lanigan")
-    (comment 2 "Surface-mount LED board")
-    (comment 4 "Released under the CERN Open Hardware Licence v1.2")
+    (date 2018-07-08)
   )
   (layers
@@
       (net 2 "Net-(D1-Pad2)"))
   )
+  (gr_line (start 157.5 116.7) (end 157.5 82.3) (layer Edge.Cuts) (width 0.15))
+  (gr_line (start 133.5 116.7) (end 133.5 82.3) (layer Edge.Cuts) (width 0.15))
   (gr_text WiLED (at 143 115.5) (layer F.SilkS)
     (effects (font (size 2 2) (thickness 0.4)) (justify right))
@@
     (effects (font (size 1.4 1.4) (thickness 0.3)) (justify right))
   )
-  (gr_line (start 158 114.5) (end 158 84.5) (angle 90) (layer Edge.Cuts) (width 0.15))
   (gr_line (start 138 119.5) (end 153 119.5) (angle 90) (layer Edge.Cuts) (width 0.15))
-  (gr_line (start 133 84.5) (end 133 114.5) (angle 90) (layer Edge.Cuts) (width 0.15))
   (gr_line (start 138 79.5) (end 153 79.5) (angle 90) (layer Edge.Cuts) (width 0.15))
-  (gr_arc (start 153 114.5) (end 158 114.5) (angle 90) (layer Edge.Cuts) (width 0.15))
-  (gr_arc (start 138 114.5) (end 138 119.5) (angle 90) (layer Edge.Cuts) (width 0.15))
-  (gr_arc (start 153 84.5) (end 153 79.5) (angle 90) (layer Edge.Cuts) (width 0.15))
-  (gr_arc (start 138 84.5) (end 133 84.5) (angle 90) (layer Edge.Cuts) (width 0.15))
+  (gr_arc (start 153 114.5) (end 157.5 116.7) (angle 63.94650469) (layer Edge.Cuts) (width 0.15))
+  (gr_arc (start 138 114.5) (end 138 119.5) (angle 63.94650743) (layer Edge.Cuts) (width 0.15))
+  (gr_arc (start 153 84.5) (end 153 79.5) (angle 63.94650743) (layer Edge.Cuts) (width 0.15))
+  (gr_arc (start 138 84.5) (end 138 79.5) (angle -63.94650743) (layer Edge.Cuts) (width 0.15))
   (segment (start 144.15 83.5) (end 139.5 83.5) (width 1.25) (layer F.Cu) (net 1))
   (segment (start 136.5 86.5) (end 136.5 88.85) (width 1.25) (layer F.Cu) (net 1))
@@
       )
     )
+  )
+  (zone (net 0) (net_name "") (layer F.Cu) (hatch edge 0.508)
+    (connect_pads (clearance 0.508))
+    (min_thickness 0.254)
+    (keepout (tracks allowed) (vias allowed) (copperpour not_allowed))
+    (fill (arc_segments 16) (thermal_gap 0.508) (thermal_bridge_width 0.508))
+    (polygon
+      (pts
+        (xy 156.9 117.6) (xy 156.9 81.4) (xy 158.1 81.4) (xy 158.1 117.6)
+      )
+    )
